Commit message: Adds working robot, and communication with ROS, additionally adds lidar model

File: description/robot.urdf.xacro (robot description, xacro)
@@ -1,4 +1,8 @@
 <?xml version="1.0"?>
-<robot xmlns:xacro="http://www.ros.org/wiki/xacro"  name="robot">
-<xacro:include filename="robot_core.xacro" />
+<robot xmlns:xacro="http://www.ros.org/wiki/xacro" name="robot">
+    <xacro:include filename="colors.xacro" />
+    <xacro:include filename="inertial_macros.xacro" />
+    <xacro:include filename="lidar.xacro" />
+    <xacro:include filename="robot_core.xacro" />
+    <xacro:include filename="gazebo_control.xacro" />
 </robot>

File: description/robot_core.xacro (robot description, xacro)
@@ -1,6 +1,4 @@
 <?xml version="1.0"?>
 <robot xmlns:xacro="http://www.ros.org/wiki/xacro">
-    <xacro:include filename="colors.xacro" />
-    <xacro:include filename="inertial_macros.xacro" />
     <link name="base_link"></link>
     <!-- CHASSIS -->
@@ -23,4 +21,5 @@
         </visual>
         <collision>
+            <origin xyz="0.15 0 0.075" />
             <geometry>
                 <box size="${chassis_width} ${chassis_length} ${chassis_height}" />
@@ -31,4 +30,8 @@
         </xacro:inertial_box>
     </link>
+    <!-- gazebo uses different materials/colors than rviz so for correct dispaly requires additional tags -->
+    <gazebo reference="chassis">
+        <material>Gazebo/White</material>
+    </gazebo>
     <!-- WHEELS -->
     <xacro:property name="wheel_mass" value="0.1" />
@@ -62,4 +65,7 @@
         </xacro:inertial_cylinder>
     </link>
+    <gazebo reference="left_wheel">
+        <material>Gazebo/Blue</material>
+    </gazebo>
     <!-- RIGHT WHEEL -->
     <joint name="right_wheel_joint" type="continuous">
@@ -87,4 +93,7 @@
         </xacro:inertial_cylinder>
     </link>
+    <gazebo reference="right_wheel">
+        <material>Gazebo/Blue</material>
+    </gazebo>
     <!-- CASTER WHEEL -->
     <xacro:property name="caster_mass" value="0.1" />
@@ -111,3 +120,8 @@
         </xacro:inertial_sphere>
     </link>
+    <gazebo reference="caster_wheel">
+        <material>Gazebo/Black</material>
+        <mu1 value="0.001" />
+        <mu2 value="0.001" />
+    </gazebo>
 </robot>
