Commit message: Adds integrated with ros camera, teleop works

File: description/colors.xacro (robot description, xacro)
@@ -7,4 +7,10 @@
         <color rgba="1 0.3 0.1 1" />
     </material>
+    <material name="red">
+        <color rgba="1 0 0 1" />
+    </material>
+    <material name="yellow">
+        <color rgba="1 1 0 1" />
+    </material>
     <material name="blue">
         <color rgba="0.2 0.2 1 1" />

File: description/lidar.xacro (robot description, xacro)
@@ -7,5 +7,5 @@
         <parent link="chassis" />
         <child link="laser_frame" />
-        <origin xyz="0.1 0 0.175" rpy="0 0 0" />
+        <origin xyz="0.1 0 0.155" rpy="0 0 0" />
     </joint>
     <link name="laser_frame">
@@ -27,4 +27,31 @@
     <gazebo reference="laser_frame">
         <material>Gazebo/Red</material>
+        <sensor name="laser" type="ray">
+            <pose> 0 0 0 0 0 0 </pose>
+            <visualize>true</visualize>
+            <update_rate>10</update_rate>
+            <!-- parameters for simulated sensor, should be as similar
+                as possible to real object-->
+            <ray>
+                <scan>
+                    <horizontal>
+                        <samples>360</samples>
+                        <min_angle>-3.14</min_angle>
+                        <max_angle>3.14</max_angle>
+                    </horizontal>
+                </scan>
+                <range>
+                    <min>0.3</min>
+                    <max>12</max>
+                </range>
+            </ray>
+            <plugin name="laser_controller" filename="libgazebo_ros_ray_sensor.so">
+                <ros>
+                    <argument>~/out:=scan</argument>
+                </ros>
+                <output_type>sensor_msgs/LaserScan</output_type>
+                <frame_name>laser_frame</frame_name>
+            </plugin>
+        </sensor>
     </gazebo>
 </robot>

File: description/robot.urdf.xacro (robot description, xacro)
@@ -3,6 +3,7 @@
     <xacro:include filename="colors.xacro" />
     <xacro:include filename="inertial_macros.xacro" />
+    <xacro:include filename="robot_core.xacro" />
     <xacro:include filename="lidar.xacro" />
-    <xacro:include filename="robot_core.xacro" />
+    <xacro:include filename="camera.xacro" />
     <xacro:include filename="gazebo_control.xacro" />
 </robot>

File: description/robot_core.xacro (robot description, xacro)
@@ -14,5 +14,5 @@
     <link name="chassis">
         <visual>
-            <origin xyz="0.15 0 0.075" rpy="0 0 0" /> <!-- przesuniecie geometrii od punktu referencyjnego -->
+            <origin xyz="${chassis_width* 0.5} 0 0${chassis_height * 0.5}" rpy="0 0 0" /> <!-- przesuniecie geometrii od punktu referencyjnego, polowa wymiarow jak rzucisz okiem-->
             <geometry>
                 <box size="${chassis_width} ${chassis_length} ${chassis_height}" />
@@ -27,5 +27,5 @@
         </collision>
         <xacro:inertial_box mass="${chassis_mass}" x="${chassis_width}" y="${chassis_length}" z="${chassis_height}">
-            <origin xyz="0.15 0 0.075" rpy="0 0 0" />
+            <origin xyz="${chassis_width* 0.5} 0 0${chassis_height * 0.5}" rpy="0 0 0" />
         </xacro:inertial_box>
     </link>
